File: roboremote/roboremote/roboremote.kicad_pcb (KiCad board)
At the start: 2 copper layers, 15 parts, among them SW1 SW_Push, SW2 SW_Push, SW3 SW_Push, SW4 SW_Push, SW5 SW_Push, U1 ESP32-C3-DevKitM-1

Commit message: pcb components layout and start journal
Parts:
- removed R7: R, Resistor_THT:R_Axial_DIN0207_L6.3mm_D2.5mm_P10.16mm_Horizontal
- removed SW5: SW_Push, MX_Solderable:MX-Solderable-1U
- U1: value ESP32-C3-DevKitM-1 -> WEMOS_C3_mini; footprint RF_Module:ESP32-C3-DevKitM-1 -> RF_Module:WEMOS_C3_mini
- moved R1 62.6 mm to (142.0, 132.1), turned to 90 degrees
- moved R2 57.5 mm to (146.1, 132.1), turned to 90 degrees
- moved SW3 53.2 mm to (177.8, 82.5)
- moved SW4 53.0 mm to (177.8, 101.6)
- moved R3 52.4 mm to (150.1, 132.1), turned to 90 degrees
- moved U1 49.4 mm to (164.1, 92.2), turned to 180 degrees
- moved R4 47.6 mm to (154.2, 132.1), turned to 90 degrees
- moved R5 42.9 mm to (158.2, 132.1), turned to 90 degrees
- moved R6 38.5 mm to (162.3, 132.1), turned to 90 degrees
- moved S2 9.69 mm to (177.8, 127.0)
- moved S1 4.05 mm to (127.0, 127.0)
- moved SW2 2.14 mm to (127.0, 101.6)
- moved SW1 2.14 mm to (127.0, 82.5)
Connections:
- R1 pad 2: D0 -> D4
- R2 pad 2: D1 -> D5
- R3 pad 2: D4 -> D8
- R4 pad 2: D2 -> D6
- R5 pad 2: D3 -> D7
- R6 pad 2: D5 -> D10
- S1 pad B2A: D0 -> D4
- S2 pad B2A: D1 -> D5
- SW1 pad 2: D2 -> D6
- SW2 pad 2: D3 -> D7
- SW3 pad 2: D4 -> D8
- SW4 pad 2: D5 -> D10
- U1 pad 1: GND -> unconnected-(U1-EN-Pad1)
- U1 pad 10: A1 -> GND
- U1 pad 12: GND -> D7
- U1 pad 13: +5V -> D8
- U1 pad 14: +5V -> D10
- U1 pad 15: GND -> unconnected-(U1-RX-Pad15)
- U1 pad 16: GND -> unconnected-(U1-TX-Pad16)
- U1 pad 2: +3V3 -> A3
- U1 pad 3: +3V3 -> A2
- U1 pad 4: A2 -> A1
- U1 pad 5: A3 -> A0
- U1 pad 6: GND -> D4
- U1 pad 7: unconnected-(U1-RST-Pad7) -> D5
- U1 pad 8: GND -> +3V3
- U1 pad 9: A0 -> +5V
