File: roboremote/roboremote/roboremote.kicad_sch (KiCad schematic)
At the start: 15 parts, among them SW1 SW_Push, SW2 SW_Push, SW3 SW_Push, SW4 SW_Push, SW5 SW_Push, U1 ESP32-C3-DevKitM-1

Commit message: pcb components layout and start journal
Parts:
- removed R7: R, Resistor_THT:R_Axial_DIN0207_L6.3mm_D2.5mm_P10.16mm_Horizontal, symbol Device:R
- removed SW5: SW_Push, MX_Solderable:MX-Solderable-1U, symbol Switch:SW_Push
- removed U1: ESP32-C3-DevKitM-1, RF_Module:ESP32-C3-DevKitM-1, symbol RF_Module:ESP32-C3-DevKitM-1
- added U1: WEMOS_C3_mini, RF_Module:WEMOS_C3_mini, symbol RF_Module:WEMOS_C3_mini
Connections:
- net D0 is gone; now on net D4: R1.2, S1.B2A (SEL-)
- net D1 is gone; now on net D5: R2.2, S2.B2A (SEL-)
- net D2 is gone; now on net D6: R4.2, SW1.2
- net +3V3: now also U1.8 (3V3)
- net +5V: now also U1.9 (VBus)
- net A0: now also U1.5 (D0)
- net A1: now also U1.4 (D1)
- net A2: now also U1.3 (D2)
- net A3: now also U1.2 (D3)
- net D4: now also U1.6 (D4); no longer R3.2, SW3.2
- net D5: now also U1.7 (D5); no longer R6.2, SW4.2
- net D6: now also U1.11 (D6)
- net GND: now also U1.10 (GND)
- net D3 renamed D7
- net D7: now also U1.12 (D7)
- new net D10: R6.2, SW4.2, U1.14 (D10)
- new net D8: R3.2, SW3.2, U1.13 (D8)
Other:
- note removed: "this is probably the wrong esp32 but ill fix it later"
